Commit message: Use the accel and brake maps measured on this vehicle
Autoware turns the controller's acceleration command into a pedal position by
looking it up in a map of the vehicle's response. The map in use was the generic
default, which describes a torque converter automatic that creeps. Its first row
claims 0.3 m/s2 at zero throttle and zero speed. A Pixkit is direct drive and
produces nothing until it is asked to, so from a standstill the controller under
commands, the speed error integrates, the throttle spikes, and the vehicle
lurches or faults. Once rolling the map is close enough that control behaves,
which is exactly the behaviour seen on the vehicle.

The calibrated maps were in the original Pixkit workspace, written over the
upstream defaults in place rather than saved under a name of their own, which is
why they were not obvious. They are labelled pix in the header, span twenty
velocity columns, and start at -0.005 m/s2 for 0.001 throttle. Recovered from
pix.zip and kept in pixkit_description/data, where they belong to the vehicle
rather than to whichever version of the converter package is installed.

The steer map stays upstream's, since convert_steer_cmd is false and the
steering PID handles it.

File: src/launcher/autoware_launch/vehicle/pixkit_launch/pixkit_description/urdf/vehicle.xacro (robot description, xacro)
@@ -6,5 +6,13 @@
   <link name="base_link">
     <visual>
-      <origin xyz="-0.25 0.0 0.1" rpy="0 0 ${pi/2.0}"/>
+      <!-- base_link is the rear axle on the ground, so the body mesh, centred on its own
+           origin, belongs at the vehicle longitudinal centre, 0.95 m ahead of it, from
+           (-rear_overhang + wheel_base + front_overhang) / 2. It was drawn at -0.25, over a
+           metre too far back, which left base_link and every pose marker drawn at it sitting
+           mid-body. Cosmetic, but it is what one judges by eye. To check, the rear wheels
+           should straddle base_link and the front wheels sit 1.9 m ahead.
+           Avoid a colon followed by a space anywhere in this file. The generated URDF is
+           passed as a parameter and parsed with YAML rules, and one breaks the whole launch. -->
+      <origin xyz="0.95 0.0 0.1" rpy="0 0 ${pi/2.0}"/>
       <geometry>
         <mesh filename="package://pixkit_description/mesh/hooke.dae" scale="0.001 0.001 0.001"/>
